Commit message: init mr_ramingo

File: urdf/lidar_gazebo_macro.xacro (robot description, xacro)
@@ -1,5 +1,5 @@
 <?xml version="1.0"?>
 <robot name="lidar_gazebo_macro" xmlns:xacro="http://www.ros.org/wiki/xacro">
-  <!--xacro:include filename="$(find mr_description)/urdf/utility_macro.xacro" /-->
+  <!--xacro:include filename="$(find mr_ramingo)/urdf/utility_macro.xacro" /-->
   <xacro:macro name="lidar_gazebo_sensor" params="parent" >
     <link name="laser_frame">
@@ -12,5 +12,5 @@
       <visual>
         <geometry>
-          <mesh filename="package://mr_description/meshes/lidar.stl" scale="0.001 0.001 0.001 "/>
+          <mesh filename="package://mr_ramingo/meshes/lidar.stl" scale="0.001 0.001 0.001 "/>
         </geometry>
         <material name="White"/>

File: urdf/mr_base_macro.xacro (robot description, xacro)
@@ -23,5 +23,5 @@
       <visual>
         <geometry>
-          <mesh filename="package://mr_description/meshes/mr_body.stl" scale="0.001 0.001 0.001 "/>
+          <mesh filename="package://mr_ramingo/meshes/mr_body.stl" scale="0.001 0.001 0.001 "/>
         </geometry>
         <material name="White"/>
@@ -44,5 +44,5 @@
       <visual>
         <geometry>
-          <mesh filename="package://mr_description/meshes/mr_wheel.stl" scale="0.001 0.001 0.001 "/>
+          <mesh filename="package://mr_ramingo/meshes/mr_wheel.stl" scale="0.001 0.001 0.001 "/>
         </geometry>
         <material name="Black"/>
@@ -51,5 +51,5 @@
       <collision>
         <geometry>
-          <mesh filename="package://mr_description/meshes/mr_wheel.stl" scale="0.001 0.001 0.001 "/>
+          <mesh filename="package://mr_ramingo/meshes/mr_wheel.stl" scale="0.001 0.001 0.001 "/>
         </geometry>
         <origin rpy="0 0 0" xyz="0 0 0"/>
@@ -66,5 +66,5 @@
       <visual>
         <geometry>
-          <mesh filename="package://mr_description/meshes/mr_wheel.stl" scale="0.001 0.001 0.001 "/>
+          <mesh filename="package://mr_ramingo/meshes/mr_wheel.stl" scale="0.001 0.001 0.001 "/>
         </geometry>
         <material name="Black"/>
@@ -73,5 +73,5 @@
       <collision>
         <geometry>
-          <mesh filename="package://mr_description/meshes/mr_wheel.stl" scale="0.001 0.001 0.001 "/>
+          <mesh filename="package://mr_ramingo/meshes/mr_wheel.stl" scale="0.001 0.001 0.001 "/>
         </geometry>
         <origin rpy="0 0 0" xyz="0 0 0"/>
