Commit message: init design

File: urdf/mr_base_macro.xacro (robot description, xacro)
@@ -25,5 +25,5 @@
           <mesh filename="package://mr_ramingo/meshes/mr_body.stl" scale="0.001 0.001 0.001 "/>
         </geometry>
-        <material name="White"/>
+        <material name="Blue"/>
         <origin rpy="0 0 0" xyz="0 0 0"/>
       </visual>
@@ -46,5 +46,5 @@
           <mesh filename="package://mr_ramingo/meshes/mr_wheel.stl" scale="0.001 0.001 0.001 "/>
         </geometry>
-        <material name="Black"/>
+        <material name="Green"/>
         <origin rpy="0 0 0" xyz="0 0 0"/>
       </visual>
@@ -68,5 +68,5 @@
           <mesh filename="package://mr_ramingo/meshes/mr_wheel.stl" scale="0.001 0.001 0.001 "/>
         </geometry>
-        <material name="Black"/>
+        <material name="Green"/>
         <origin rpy="0 0 0" xyz="0 0 0"/>
       </visual>

File: urdf/utility_macro.xacro (robot description, xacro)
@@ -18,4 +18,7 @@
     <color rgba="0.0 0.0 0.8 1.0"/>
   </material>
+  <material name="Green">
+    <color rgba="0.0 0.8 0.0 1.0"/>
+  </material>
   <xacro:macro name="cylinder_inertia" params="m r h">
     <inertia  ixx="${m*(3*r*r+h*h)/12}" ixy = "0" ixz = "0"
