Commit message: robot si muove con rqt

File: urdf/mr.xacro (robot description, xacro)
@@ -2,5 +2,149 @@
 <robot name="mobile_robot" xmlns:xacro="http://ros.org/wiki/xacro">
   <xacro:include filename="$(find mr_ramingo)/urdf/mr_base_macro.xacro" />
-  <!-- Diff Drive Robot Base  -->
+  <xacro:property name="LIDAR" value="True"/>
+  <!--Actual body/chassis of the robot
+	<link name="base_link">
+		<inertial>
+				<inertia ixx="1.0" ixy="0.0" ixz="0.0" iyy="1.0" iyz="0.0" izz="1.0"/>
+			<mass value="${base_mass}" />
+			<origin xyz="0 0 0" />
+			<cylinder_inertia  m="${base_mass}" r="${base_radius}" h="${base_height}" />
+		</inertial>
+		<visual>
+			<origin xyz="0 0 0" rpy="0 0 0" />
+			<geometry>
+				<cylinder length="${base_height}" radius="${base_radius}" />
+			</geometry>
+			<material name="White" />
+		</visual>
+		<collision>
+			<origin xyz="0 0 0" rpy="0 0 0 " />
+			<geometry>
+				<cylinder length="${base_height}" radius="${base_radius}" />
+			</geometry>
+		</collision>
+	</link>
+-->
+	<link name="sensor_link">
+		<!--
+    <collision>
+      <origin xyz="0 0 0.05" rpy="0 0 0"/>
+      <geometry>
+        <box size="0.1 0.1 0.1"/>
+      </geometry>
+    </collision>
+		-->
+    <visual>
+      <origin xyz="0 0 0.05" rpy="0 0 0"/>
+      <geometry>
+        <box size="0.1 0.1 0.1"/>
+      </geometry>
+      <material name="orange"/>
+    </visual>
+		<!--
+    <inertial>
+      <origin xyz="0 0 1" rpy="0 0 0"/>
+      <mass value="1"/>
+      <inertia
+        ixx="1.0" ixy="0.0" ixz="0.0"
+        iyy="1.0" iyz="0.0"
+        izz="1.0"/>
+    </inertial>
+		-->
+  </link>
+	<joint name="sensor_joint" type="fixed">
+		<parent link="base_link" />
+		<child link="sensor_link" />
+		<origin xyz="0.0 0.0 0.1" rpy="0 0 0"/>
+	</joint>
+<!--
+	<xacro:caster_joint
+		name="caster_front_link"
+		parent="base_link"
+		child="caster_front_link">
+		<origin xyz="0.115 0.0 0.007" rpy="${-M_PI/2} 0 0"/>
+	</xacro:caster_joint>
+	<xacro:caster_link
+		name="caster_front_link">
+			<origin xyz="0 0.02 0" rpy="${M_PI/2} 0 0" />
+	</xacro:caster_link>
+	<xacro:caster_joint
+		name="caster_back_joint"
+		parent="base_link"
+		child="caster_back_link">
+		<origin xyz="-0.135 0.0 0.009" rpy="${-M_PI/2} 0 0"/>
+	</xacro:caster_joint>
+	<xacro:caster_link
+		name="caster_back_link">
+			<origin xyz="0.02 0.02 0 " rpy="${M_PI/2} 0 0" />
+	</xacro:caster_link>
+-->
+	<!--
+	<xacro:wheel fb="front" lr="right" parent="base_link" translateX="0" translateY="0.5" flipY="1"/>
+	<xacro:wheel fb="front" lr="left" parent="base_link" translateX="0" translateY="-0.5" flipY="1"/>
+	<xacro:wheel fb="front" lr="right" parent="base_link" translateX="0" translateY="-0.5" flipY="1"/>
+	<xacro:wheel fb="front" lr="left" parent="base_link" translateX="0" translateY="0.5" flipY="1"/>
+  -->
+  <!-- Differential drive controller  -->
+  <gazebo>
+    <plugin name="mr_ramingo_drive_controller" filename="libgazebo_ros_diff_drive.so">
+      <legacyMode>true</legacyMode>
+      <rosDebugLevel>Debug</rosDebugLevel>
+      <publishWheelTF>false</publishWheelTF>
+      <robotNamespace>/</robotNamespace>
+      <publishTf>1</publishTf>
+      <publishWheelJointState>false</publishWheelJointState>
+      <alwaysOn>true</alwaysOn>
+      <updateRate>100.0</updateRate>
+      <leftJoint>left_wheel_joint</leftJoint>
+      <rightJoint>right_wheel_joint</rightJoint>
+      <wheelSeparation>${2*base_radius}</wheelSeparation>
+      <wheelDiameter>${2*wheel_radius}</wheelDiameter>
+      <broadcastTF>1</broadcastTF>
+      <wheelTorque>30</wheelTorque>
+      <wheelAcceleration>1.8</wheelAcceleration>
+      <commandTopic>cmd_vel</commandTopic>
+      <odometryFrame>odom</odometryFrame>
+      <odometryTopic>odom</odometryTopic>
+      <robotBaseFrame>base_link</robotBaseFrame>
+    </plugin>
+  </gazebo>
+  <xacro:if value="${LIDAR}" >
+    <gazebo reference="base_link">
+        <sensor type="ray" name="laser">
+        <pose>0 0 0.1 0 0 0</pose>
+        <visualize>true</visualize>
+        <update_rate>40</update_rate>
+        <ray>
+          <scan>
+            <horizontal>
+              <samples>720</samples>
+              <resolution>1</resolution>
+              <min_angle>-1.57</min_angle>
+              <max_angle>1.57</max_angle>
+            </horizontal>
+          </scan>
+          <range>
+            <min>0.2</min>
+            <max>30.0</max>
+            <resolution>0.01</resolution>
+          </range>
+          <noise>
+            <type>gaussian</type>
+            <!-- Noise parameters based on published spec for Hokuyo laser
+                achieving "+-30mm" accuracy at range < 10m.  A mean of 0.0m and
+                stddev of 0.01m will put 99.7% of samples within 0.03m of the true
+                reading. -->
+            <mean>0.0</mean>
+            <stddev>0.01</stddev>
+          </noise>
+        </ray>
+        <plugin name="gazebo_ros_head_hokuyo_controller" filename="libgazebo_ros_laser.so">
+          <topicName>/laser/scan</topicName>
+          <frameName>base_link</frameName>
+        </plugin>
+      </sensor>
+    </gazebo>
+	</xacro:if>
   <xacro:mr_base />
 </robot>

Commit message: cancellazione commenti

File: urdf/mr.xacro (robot description, xacro)
@@ -3,27 +3,4 @@
   <xacro:include filename="$(find mr_ramingo)/urdf/mr_base_macro.xacro" />
   <xacro:property name="LIDAR" value="True"/>
-  <!--Actual body/chassis of the robot
-	<link name="base_link">
-		<inertial>
-				<inertia ixx="1.0" ixy="0.0" ixz="0.0" iyy="1.0" iyz="0.0" izz="1.0"/>
-			<mass value="${base_mass}" />
-			<origin xyz="0 0 0" />
-			<cylinder_inertia  m="${base_mass}" r="${base_radius}" h="${base_height}" />
-		</inertial>
-		<visual>
-			<origin xyz="0 0 0" rpy="0 0 0" />
-			<geometry>
-				<cylinder length="${base_height}" radius="${base_radius}" />
-			</geometry>
-			<material name="White" />
-		</visual>
-		<collision>
-			<origin xyz="0 0 0" rpy="0 0 0 " />
-			<geometry>
-				<cylinder length="${base_height}" radius="${base_radius}" />
-			</geometry>
-		</collision>
-	</link>
--->
 	<link name="sensor_link">
 		<!--
@@ -58,32 +35,4 @@
 		<origin xyz="0.0 0.0 0.1" rpy="0 0 0"/>
 	</joint>
-<!--
-	<xacro:caster_joint
-		name="caster_front_link"
-		parent="base_link"
-		child="caster_front_link">
-		<origin xyz="0.115 0.0 0.007" rpy="${-M_PI/2} 0 0"/>
-	</xacro:caster_joint>
-	<xacro:caster_link
-		name="caster_front_link">
-			<origin xyz="0 0.02 0" rpy="${M_PI/2} 0 0" />
-	</xacro:caster_link>
-	<xacro:caster_joint
-		name="caster_back_joint"
-		parent="base_link"
-		child="caster_back_link">
-		<origin xyz="-0.135 0.0 0.009" rpy="${-M_PI/2} 0 0"/>
-	</xacro:caster_joint>
-	<xacro:caster_link
-		name="caster_back_link">
-			<origin xyz="0.02 0.02 0 " rpy="${M_PI/2} 0 0" />
-	</xacro:caster_link>
--->
-	<!--
-	<xacro:wheel fb="front" lr="right" parent="base_link" translateX="0" translateY="0.5" flipY="1"/>
-	<xacro:wheel fb="front" lr="left" parent="base_link" translateX="0" translateY="-0.5" flipY="1"/>
-	<xacro:wheel fb="front" lr="right" parent="base_link" translateX="0" translateY="-0.5" flipY="1"/>
-	<xacro:wheel fb="front" lr="left" parent="base_link" translateX="0" translateY="0.5" flipY="1"/>
-  -->
   <!-- Differential drive controller  -->
   <gazebo>

Commit message: pulizia

File: urdf/mr.xacro (robot description, xacro)
@@ -2,6 +2,6 @@
 <robot name="mobile_robot" xmlns:xacro="http://ros.org/wiki/xacro">
   <xacro:include filename="$(find mr_ramingo)/urdf/mr_base_macro.xacro" />
-  <xacro:include filename="$(find mr_ramingo)/urdf/camera.xacro" />
-  <xacro:property name="LIDAR" value="True"/>
+  <!--xacro:include filename="$(find mr_ramingo)/urdf/lidar_camera_gazebo.xacro" /-->
+  <xacro:include filename="$(find mr_ramingo)/urdf/lidar.xacro"/>
 	<link name="camera_link">
 		<!--
@@ -36,18 +36,4 @@
 		<origin xyz="0.11 0.0 0.0" rpy="0 0 0"/>
 	</joint>
-	<link name="laser">
-    <visual>
-      <origin xyz="0 0 0" rpy="0 0 0"/>
-      <geometry>
-        <box size="0.05 0.05 0.05"/>
-      </geometry>
-      <material name="yellow"/>
-    </visual>
-  </link>
-	<joint name="laser_joint" type="fixed">
-		<parent link="base_link" />
-		<child link="laser" />
-		<origin xyz="0.0 0.0 0.15" rpy="0 0 0"/>
-	</joint>
   <!-- Differential drive controller  -->
   <gazebo>
@@ -74,41 +60,5 @@
     </plugin>
   </gazebo>
-  <xacro:if value="${LIDAR}" >
-    <gazebo reference="base_link">
-        <sensor type="ray" name="laser">
-        <pose>0 0 0.1 0 0 0</pose>
-        <visualize>true</visualize>
-        <update_rate>40</update_rate>
-        <ray>
-          <scan>
-            <horizontal>
-              <samples>720</samples>
-              <resolution>1</resolution>
-              <min_angle>-1.57</min_angle>
-              <max_angle>1.57</max_angle>
-            </horizontal>
-          </scan>
-          <range>
-            <min>0.2</min>
-            <max>30.0</max>
-            <resolution>0.01</resolution>
-          </range>
-          <noise>
-            <type>gaussian</type>
-            <!-- Noise parameters based on published spec for Hokuyo laser
-                achieving "+-30mm" accuracy at range < 10m.  A mean of 0.0m and
-                stddev of 0.01m will put 99.7% of samples within 0.03m of the true
-                reading. -->
-            <mean>0.0</mean>
-            <stddev>0.01</stddev>
-          </noise>
-        </ray>
-        <plugin name="gazebo_ros_head_hokuyo_controller" filename="libgazebo_ros_laser.so">
-          <topicName>/laser/scan</topicName>
-          <frameName>base_link</frameName>
-        </plugin>
-      </sensor>
-    </gazebo>
-	</xacro:if>
   <xacro:mr_base />
+  <xacro:lidar />
 </robot>
