Commit message: pulizia codice

File: urdf/lidar_camera_gazebo.xacro (robot description, xacro)
@@ -16,10 +16,10 @@
 		<parent link="base_link" />
 		<child link="laser" />
-		<origin xyz="0.0 0.0 0.15" rpy="0 0 0"/>
+		<origin xyz="0.0 0.0 0.125" rpy="0 0 0"/>
 	</joint>
   <xacro:if value="${LIDAR}" >
       <gazebo reference="base_link">
           <sensor type="ray" name="laser">
-          <pose>0 0 0.1 0 0 0</pose>
+          <pose>0 0 0.127 0 0 0</pose>
           <visualize>true</visualize>
           <update_rate>40</update_rate>

File: urdf/mr.xacro (robot description, xacro)
@@ -2,38 +2,7 @@
 <robot name="mobile_robot" xmlns:xacro="http://ros.org/wiki/xacro">
   <xacro:include filename="$(find mr_ramingo)/urdf/mr_base_macro.xacro" />
-  <!--xacro:include filename="$(find mr_ramingo)/urdf/lidar_camera_gazebo.xacro" /-->
-  <xacro:include filename="$(find mr_ramingo)/urdf/lidar.xacro"/>
-	<link name="camera_link">
-		<!--
-    <collision>
-      <origin xyz="0 0 0.05" rpy="0 0 0"/>
-      <geometry>
-        <box size="0.1 0.1 0.1"/>
-      </geometry>
-    </collision>
-		-->
-    <visual>
-      <origin xyz="0 0 0" rpy="0 0 0"/>
-      <geometry>
-        <box size="0.01 0.02 0.02"/>
-      </geometry>
-      <material name="orange"/>
-    </visual>
-		<!--
-    <inertial>
-      <origin xyz="0 0 1" rpy="0 0 0"/>
-      <mass value="1"/>
-      <inertia
-        ixx="1.0" ixy="0.0" ixz="0.0"
-        iyy="1.0" iyz="0.0"
-        izz="1.0"/>
-    </inertial>
-		-->
-  </link>
-	<joint name="camera_joint" type="fixed">
-		<parent link="base_link" />
-		<child link="camera_link" />
-		<origin xyz="0.11 0.0 0.0" rpy="0 0 0"/>
-	</joint>
+  <xacro:include filename="$(find mr_ramingo)/urdf/lidar_camera_gazebo.xacro" />
+  <!--xacro:include filename="$(find mr_ramingo)/urdf/lidar.xacro"/>
+  <xacro:include filename="$(find mr_ramingo)/urdf/camera.xacro"/-->
   <!-- Differential drive controller  -->
   <gazebo>
@@ -60,5 +29,6 @@
     </plugin>
   </gazebo>
+  <!--xacro:camera />
+  <xacro:lidar /-->
   <xacro:mr_base />
-  <xacro:lidar />
 </robot>
