Commit message: config lidar

File: urdf/camera.xacro (robot description, xacro)
@@ -1,6 +1,5 @@
 <?xml version="1.0"?>
 <robot name="sensor" xmlns:xacro="http://www.ros.org/wiki/xacro">
-  <gazebo reference="sensor_link">
-    <pose>0 1 0.05 0 0 0</pose>
+  <gazebo reference="camera_link">
     <sensor type="camera" name="camera1">
       <update_rate>30.0</update_rate>

File: urdf/mr.xacro (robot description, xacro)
@@ -4,5 +4,5 @@
   <xacro:include filename="$(find mr_ramingo)/urdf/camera.xacro" />
   <xacro:property name="LIDAR" value="True"/>
-	<link name="sensor_link">
+	<link name="camera_link">
 		<!--
     <collision>
@@ -14,7 +14,7 @@
 		-->
     <visual>
-      <origin xyz="0 0 0.05" rpy="0 0 0"/>
+      <origin xyz="0 0 0" rpy="0 0 0"/>
       <geometry>
-        <box size="0.1 0.1 0.1"/>
+        <box size="0.01 0.02 0.02"/>
       </geometry>
       <material name="orange"/>
@@ -31,8 +31,22 @@
 		-->
   </link>
-	<joint name="sensor_joint" type="fixed">
+	<joint name="camera_joint" type="fixed">
 		<parent link="base_link" />
-		<child link="sensor_link" />
-		<origin xyz="0.0 0.0 0.1" rpy="0 0 0"/>
+		<child link="camera_link" />
+		<origin xyz="0.11 0.0 0.0" rpy="0 0 0"/>
+	</joint>
+	<link name="laser">
+    <visual>
+      <origin xyz="0 0 0" rpy="0 0 0"/>
+      <geometry>
+        <box size="0.05 0.05 0.05"/>
+      </geometry>
+      <material name="yellow"/>
+    </visual>
+  </link>
+	<joint name="laser_joint" type="fixed">
+		<parent link="base_link" />
+		<child link="laser" />
+		<origin xyz="0.0 0.0 0.15" rpy="0 0 0"/>
 	</joint>
   <!-- Differential drive controller  -->
@@ -45,5 +59,4 @@
       <publishTf>0</publishTf>
       <publishWheelJointState>false</publishWheelJointState>
-      <!--publishOdomTF>false</publishOdomTF-->
       <alwaysOn>true</alwaysOn>
       <updateRate>100.0</updateRate>

Commit message: goal quasi pronto

File: urdf/camera.xacro (robot description, xacro)
@@ -33,5 +33,5 @@
 		<parent link="base_link" />
 		<child link="camera_link" />
-		<origin xyz="0.11 0.0 0.0" rpy="0 0 0"/>
+		<origin xyz="0.11 0.0 0.0" rpy="0 1.57 0"/>
 	</joint>
   </xacro:macro>

File: urdf/lidar_camera_gazebo.xacro (robot description, xacro)
@@ -2,5 +2,5 @@
 <robot name="sensor" xmlns:xacro="http://www.ros.org/wiki/xacro">
   <xacro:property name="LIDAR" value="True"/>
-  <xacro:property name="CAMERA" value="True"/>
+  <xacro:property name="CAMERA" value="False"/>
   <!--TF LiDAR real -->
 	<link name="laser">

Commit message: prova1 sul robot

File: urdf/camera.xacro (robot description, xacro)
@@ -35,4 +35,36 @@
 		<origin xyz="0.11 0.0 0.0" rpy="0 1.57 0"/>
 	</joint>
+  <link name="fix_camera_link">
+		<!--
+    <collision>
+      <origin xyz="0 0 0.05" rpy="0 0 0"/>
+      <geometry>
+        <box size="0.1 0.1 0.1"/>
+      </geometry>
+    </collision>
+		-->
+    <visual>
+      <origin xyz="0 0 0" rpy="0 0 0"/>
+      <geometry>
+        <box size="0.01 0.02 0.02"/>
+      </geometry>
+      <material name="orange"/>
+    </visual>
+		<!--
+    <inertial>
+      <origin xyz="0 0 1" rpy="0 0 0"/>
+      <mass value="1"/>
+      <inertia
+        ixx="1.0" ixy="0.0" ixz="0.0"
+        iyy="1.0" iyz="0.0"
+        izz="1.0"/>
+    </inertial>
+		-->
+  </link>
+	<joint name="fix_camera_joint" type="fixed">
+		<parent link="camera_link" />
+		<child link="fix_camera_link" />
+		<origin xyz="0 0.0 0.0" rpy="0 -1.57 0"/>
+	</joint>
   </xacro:macro>
 </robot>

File: urdf/lidar_camera_gazebo.xacro (robot description, xacro)
@@ -2,5 +2,5 @@
 <robot name="sensor" xmlns:xacro="http://www.ros.org/wiki/xacro">
   <xacro:property name="LIDAR" value="True"/>
-  <xacro:property name="CAMERA" value="False"/>
+  <xacro:property name="CAMERA" value="True"/>
   <!--TF LiDAR real -->
 	<link name="laser">
@@ -57,5 +57,5 @@
   <!--Config Camera Gazebo-->
     <xacro:if value="${CAMERA}" >
-      <gazebo reference="camera_link">
+      <gazebo reference="fix_camera_link">
         <sensor type="camera" name="camera1">
           <update_rate>30.0</update_rate>

File: urdf/mr.xacro (robot description, xacro)
@@ -3,6 +3,6 @@
   <xacro:include filename="$(find mr_ramingo)/urdf/mr_base_macro.xacro" />
   <xacro:include filename="$(find mr_ramingo)/urdf/lidar_camera_gazebo.xacro" />
-  <!--xacro:include filename="$(find mr_ramingo)/urdf/lidar.xacro"/-->
-  <xacro:include filename="$(find mr_ramingo)/urdf/camera.xacro"/>
+  <xacro:include filename="$(find mr_ramingo)/urdf/lidar.xacro"/>
+  <!--xacro:include filename="$(find mr_ramingo)/urdf/camera.xacro"/-->
   <!-- Differential drive controller  -->
   <gazebo>

Commit message: unico launch real/gazebo

File: urdf/camera.xacro (robot description, xacro)
@@ -17,5 +17,5 @@
         <box size="0.01 0.02 0.02"/>
       </geometry>
-      <material name="orange"/>
+      <material name="Red"/>
     </visual>
 		<!--
@@ -49,5 +49,5 @@
         <box size="0.01 0.02 0.02"/>
       </geometry>
-      <material name="orange"/>
+      <material name="Red"/>
     </visual>
 		<!--

File: urdf/lidar_camera_gazebo.xacro (robot description, xacro)
@@ -3,5 +3,5 @@
   <xacro:property name="LIDAR" value="True"/>
   <xacro:property name="CAMERA" value="True"/>
-  <!--TF LiDAR real -->
+  <!--TF LiDAR real >
 	<link name="laser">
     <visual>
@@ -17,5 +17,5 @@
 		<child link="laser" />
 		<origin xyz="0.0 0.0 0.125" rpy="0 0 0"/>
-	</joint>
+	</joint-->
   <xacro:if value="${LIDAR}" >
       <gazebo reference="base_link">

File: urdf/mr.xacro (robot description, xacro)
@@ -1,6 +1,10 @@
 <?xml version="1.0"?>
 <robot name="mobile_robot" xmlns:xacro="http://ros.org/wiki/xacro">
+  <!--Set False if in real mode-->
+  <xacro:arg name="MR_GAZEBO" default="True"/>
   <xacro:include filename="$(find mr_ramingo)/urdf/mr_base_macro.xacro" />
-  <!--xacro:include filename="$(find mr_ramingo)/urdf/lidar_camera_gazebo.xacro" /-->
+  <xacro:if value="$(arg MR_GAZEBO)" >
+    <xacro:include filename="$(find mr_ramingo)/urdf/lidar_camera_gazebo.xacro" />
+  </xacro:if>
   <xacro:include filename="$(find mr_ramingo)/urdf/lidar.xacro"/>
   <xacro:include filename="$(find mr_ramingo)/urdf/camera.xacro"/>

Commit message: aggiustato frame aruco

File: urdf/camera.xacro (robot description, xacro)
@@ -35,13 +35,5 @@
 		<origin xyz="0.11 0.0 0.0" rpy="0 1.57 0"/>
 	</joint>
-  <link name="fix_camera_link">
-		<!--
-    <collision>
-      <origin xyz="0 0 0.05" rpy="0 0 0"/>
-      <geometry>
-        <box size="0.1 0.1 0.1"/>
-      </geometry>
-    </collision>
-		-->
+  <link name="gazebo_camera_link">
     <visual>
       <origin xyz="0 0 0" rpy="0 0 0"/>
@@ -51,19 +43,23 @@
       <material name="Red"/>
     </visual>
-		<!--
-    <inertial>
-      <origin xyz="0 0 1" rpy="0 0 0"/>
-      <mass value="1"/>
-      <inertia
-        ixx="1.0" ixy="0.0" ixz="0.0"
-        iyy="1.0" iyz="0.0"
-        izz="1.0"/>
-    </inertial>
-		-->
   </link>
-	<joint name="fix_camera_joint" type="fixed">
+	<joint name="gazebo_camera_joint" type="fixed">
 		<parent link="camera_link" />
-		<child link="fix_camera_link" />
+		<child link="gazebo_camera_link" />
 		<origin xyz="0 0.0 0.0" rpy="0 -1.57 0"/>
+	</joint>
+  <link name="gazebo_aruco_camera_link">
+    <visual>
+      <origin xyz="0 0 0" rpy="0 0 0"/>
+      <geometry>
+        <box size="0.01 0.02 0.02"/>
+      </geometry>
+      <material name="Red"/>
+    </visual>
+  </link>
+	<joint name="gazebo_aruco_camera_joint" type="fixed">
+		<parent link="camera_link" />
+		<child link="gazebo_aruco_camera_link" />
+		<origin xyz="0 0.0 0.0" rpy="0 0 -1.57"/>
 	</joint>
   </xacro:macro>

File: urdf/lidar_camera_gazebo.xacro (robot description, xacro)
@@ -57,5 +57,5 @@
   <!--Config Camera Gazebo-->
     <xacro:if value="${CAMERA}" >
-      <gazebo reference="fix_camera_link">
+      <gazebo reference="gazebo_camera_link">
         <sensor type="camera" name="camera1">
           <update_rate>30.0</update_rate>

Commit message: definitivo

File: urdf/camera.xacro (robot description, xacro)
@@ -35,5 +35,5 @@
 		<origin xyz="0.11 0.0 0.0" rpy="0 1.57 0"/>
 	</joint>
-  <link name="gazebo_camera_link">
+  <link name="real_camera_link">
     <visual>
       <origin xyz="0 0 0" rpy="0 0 0"/>
@@ -44,22 +44,8 @@
     </visual>
   </link>
-	<joint name="gazebo_camera_joint" type="fixed">
+	<joint name="real_camera_joint" type="fixed">
 		<parent link="camera_link" />
-		<child link="gazebo_camera_link" />
-		<origin xyz="0 0.0 0.0" rpy="0 -1.57 0"/>
-	</joint>
-  <link name="gazebo_aruco_camera_link">
-    <visual>
-      <origin xyz="0 0 0" rpy="0 0 0"/>
-      <geometry>
-        <box size="0.01 0.02 0.02"/>
-      </geometry>
-      <material name="Red"/>
-    </visual>
-  </link>
-	<joint name="gazebo_aruco_camera_joint" type="fixed">
-		<parent link="camera_link" />
-		<child link="gazebo_aruco_camera_link" />
-		<origin xyz="0 0.0 0.0" rpy="0 0 -1.57"/>
+		<child link="real_camera_link" />
+		<origin xyz="0 0.0 0.0" rpy="0 0 1.57"/>
 	</joint>
   </xacro:macro>

File: urdf/lidar.xacro (robot description, xacro)
@@ -28,5 +28,5 @@
       <parent link="base_link"/>
       <child link="laser"/>
-      <origin rpy="0 0 0" xyz="0.0 0.0 0.151"/>
+      <origin rpy="3.14 0 3.14" xyz="0.0 0.0 0.151"/>
     </joint>
   </xacro:macro>

File: urdf/lidar_camera_gazebo.xacro (robot description, xacro)
@@ -3,4 +3,32 @@
   <xacro:property name="LIDAR" value="True"/>
   <xacro:property name="CAMERA" value="True"/>
+  <link name="gazebo_camera_link">
+    <visual>
+      <origin xyz="0 0 0" rpy="0 0 0"/>
+      <geometry>
+        <box size="0.01 0.02 0.02"/>
+      </geometry>
+      <material name="Red"/>
+    </visual>
+  </link>
+	<joint name="gazebo_camera_joint" type="fixed">
+		<parent link="camera_link" />
+		<child link="gazebo_camera_link" />
+		<origin xyz="0 0.0 0.0" rpy="0 -1.57 0"/>
+	</joint>
+  <link name="gazebo_aruco_camera_link">
+    <visual>
+      <origin xyz="0 0 0" rpy="0 0 0"/>
+      <geometry>
+        <box size="0.01 0.02 0.02"/>
+      </geometry>
+      <material name="Red"/>
+    </visual>
+  </link>
+	<joint name="gazebo_aruco_camera_joint" type="fixed">
+		<parent link="camera_link" />
+		<child link="gazebo_aruco_camera_link" />
+		<origin xyz="0 0.0 0.0" rpy="0 0 -1.57"/>
+	</joint>
   <!--TF LiDAR real >
 	<link name="laser">

File: urdf/mr.xacro (robot description, xacro)
@@ -2,5 +2,5 @@
 <robot name="mobile_robot" xmlns:xacro="http://ros.org/wiki/xacro">
   <!--Set False if in real mode-->
-  <xacro:arg name="MR_GAZEBO" default="True"/>
+  <xacro:arg name="MR_GAZEBO" default="False"/>
   <xacro:include filename="$(find mr_ramingo)/urdf/mr_base_macro.xacro" />
   <xacro:if value="$(arg MR_GAZEBO)" >

Commit message: pulizia

File: urdf/camera.xacro (robot description, xacro)
@@ -35,5 +35,5 @@
 		<origin xyz="0.11 0.0 0.0" rpy="0 1.57 0"/>
 	</joint>
-  <link name="real_camera_link">
+  <link name="aruco_camera_link">
     <visual>
       <origin xyz="0 0 0" rpy="0 0 0"/>
@@ -44,7 +44,7 @@
     </visual>
   </link>
-	<joint name="real_camera_joint" type="fixed">
+	<joint name="aruco_camera_joint" type="fixed">
 		<parent link="camera_link" />
-		<child link="real_camera_link" />
+		<child link="aruco_camera_link" />
 		<origin xyz="0 0.0 0.0" rpy="0 0 1.57"/>
 	</joint>

File: urdf/lidar.xacro (robot description, xacro)
@@ -15,5 +15,5 @@
         </geometry>
         <material name="White"/>
-        <origin rpy="0 0 ${-M_PI_2}" xyz="0.0 0.0 -0.031"/>
+        <origin rpy="3.14 0 ${-M_PI_2}" xyz="0.0 0.0 -0.031"/>
       </visual>
       <collision>
@@ -22,5 +22,5 @@
           <cylinder length="0.04" radius="0.037" />
         </geometry>
-        <origin rpy="0 0 0" xyz="0.0 0.0 -0.031"/>
+        <origin rpy="3.14 0 0" xyz="0.0 0.0 -0.031"/>
       </collision>
     </link>
@@ -28,5 +28,5 @@
       <parent link="base_link"/>
       <child link="laser"/>
-      <origin rpy="3.14 0 3.14" xyz="0.0 0.0 0.151"/>
+      <origin rpy="3.14 0 3.14" xyz="0.0 0.0 0.095"/>
     </joint>
   </xacro:macro>

File: urdf/lidar_camera_gazebo.xacro (robot description, xacro)
@@ -49,5 +49,5 @@
       <gazebo reference="base_link">
           <sensor type="ray" name="laser">
-          <pose>0 0 0.127 0 0 0</pose>  <!--Melania z = 0.02 -->
+          <pose>0 0 0.02 0 0 0</pose>  <!--Melania z = 0.02  default 0.127-->
           <visualize>true</visualize>
           <update_rate>40</update_rate>
